File: Header_Board.sch (KiCad schematic (older format))
At the start: 2 parts, among them P1 CONN_02X26, P2 CONN_02X26

Commit message: Add files via upload
Parts:
- added J1, J2: Conn_Coaxial, Connectors:SMA_SMD_Jack_Straight, symbol Conn_Coaxial
- added P3: CONN_02X30, Connectors_Samtec:MECF-30-01-NP-L-DV-WT_Socket, symbol CONN_02X30
- added U1, U10, U12: TAMP_1512GLN+, Project:TAMP-1512GLN+, symbol TAMP_1512GLN+
- added U11, U13, U14, U15, U17, U18, U3, U4, U5, U6, U7, U9: LAT, Project:LAT_1+, symbol LAT
- added U16, U2, U8: CBP-1400E+, Project:CBP-1400E+, symbol CBP-1400E+
- P1, P2: footprint (none) -> Project:CSK_Header
Connections:
- net +3V3: now also P3.11 (P11), P3.14 (P14), P3.2 (P2), P3.33 (P33), P3.36 (P36), P3.53 (P53), P3.56 (P56)
- net +5V: now also P3.3 (P3), P3.57 (P57), U1.5 (5V), U10.5 (5V), U12.5 (5V)
- net GND: now also J1.2 (Ext), J2.2 (Ext), P3.1 (P1), P3.12 (P12), P3.13 (P13), P3.16 (P16), P3.17 (P17), P3.20 (P20), P3.23 (P23), P3.26 (P26), P3.27 (P27), P3.30 (P30), P3.31 (P31), P3.34 (P34), P3.35 (P35), P3.38 (P38), P3.39 (P39), P3.4 (P4), P3.42 (P42), P3.43 (P43), P3.46 (P46), P3.47 (P47), P3.5 (P5), P3.50 (P50), P3.51 (P51), P3.54 (P54), P3.55 (P55), P3.58 (P58), P3.59 (P59), P3.8 (P8), P3.9 (P9), U1.1 (GND), U1.10 (GND), U1.11 (GND), U1.3 (GND), U1.4 (GND), U1.6 (GND), U1.8 (GND), U1.9 (GND), U10.1 (GND), U10.10 (GND), U10.11 (GND), U10.3 (GND), U10.4 (GND), U10.6 (GND), U10.8 (GND), U10.9 (GND), U11.1 (GND), U11.3 (GND), U12.1 (GND), U12.10 (GND), U12.11 (GND), U12.3 (GND), U12.4 (GND), U12.6 (GND), U12.8 (GND), U12.9 (GND), U13.1 (GND), U13.3 (GND), U14.1 (GND), U14.3 (GND), U15.1 (GND), U15.3 (GND), U16.10 (GND), U16.12 (GND), U16.13 (GND), U16.14 (GND), U16.15 (GND), U16.16 (GND), U16.2 (GND), U16.3 (GND), U16.4 (GND), U16.5 (GND), U16.6 (GND), U16.7 (GND), U16.8 (GND), U16.9 (GND), U17.1 (GND), U17.3 (GND), U18.1 (GND), U18.3 (GND), U2.10 (GND), U2.12 (GND), U2.13 (GND), U2.14 (GND), U2.15 (GND), U2.16 (GND), U2.2 (GND), U2.3 (GND), U2.4 (GND), U2.5 (GND), U2.6 (GND), U2.7 (GND), U2.8 (GND), U2.9 (GND), U3.1 (GND), U3.3 (GND), U4.1 (GND), U4.3 (GND), U5.1 (GND), U5.3 (GND), U6.1 (GND), U6.3 (GND), U7.1 (GND), U7.3 (GND), U8.10 (GND), U8.12 (GND), U8.13 (GND), U8.14 (GND), U8.15 (GND), U8.16 (GND), U8.2 (GND), U8.3 (GND), U8.4 (GND), U8.5 (GND), U8.6 (GND), U8.7 (GND), U8.8 (GND), U8.9 (GND), U9.1 (GND), U9.3 (GND)
- net SPI2_MISO: now also P3.15 (P15)
- net SPI2_MOSI: now also P3.18 (P18)
- net SPI2_SCK: now also P3.19 (P19)
- net SYS_SCL: now also P3.7 (P7)
- net SYS_SDA: now also P3.10 (P10)
- net SYS_SPI_MISO: now also P3.37 (P37)
- net SYS_SPI_MOSI: now also P3.40 (P40)
- net SYS_SPI_SCK: now also P3.41 (P41)
- new net: J1.1 (In), U2.1 (RF_IN)
- new net: J2.1 (In), U12.7 (RF_OUT)
- new net: U14.2 (RF_OUT), U8.1 (RF_IN)
- new net: U10.7 (RF_OUT), U14.4 (RF_IN)
- new net: U3.4 (RF_IN), U4.2 (RF_OUT)
- new net: U4.4 (RF_IN), U8.11 (RF_OUT)
- new net: U1.2 (RF_IN), U3.2 (RF_OUT)
- new net: U5.2 (RF_OUT), U6.4 (RF_IN)
- new net: U1.7 (RF_OUT), U5.4 (RF_IN)
- new net: U6.2 (RF_OUT), U7.4 (RF_IN)
- new net: U7.2 (RF_OUT), U9.4 (RF_IN)
- new net: U11.4 (RF_IN), U9.2 (RF_OUT)
- new net: U11.2 (RF_OUT), U13.4 (RF_IN)
- new net: U13.2 (RF_OUT), U16.1 (RF_IN)
- new net: U17.4 (RF_IN), U18.2 (RF_OUT)
- new net: U16.11 (RF_OUT), U18.4 (RF_IN)
- new net: U15.4 (RF_IN), U17.2 (RF_OUT)
- new net: U12.2 (RF_IN), U15.2 (RF_OUT)
- new net: U10.2 (RF_IN), U2.11 (RF_OUT)
- new net +12V: P3.6 (P6), P3.60 (P60)
- new net GPIO_10: P3.49 (P49)
- new net GPIO_11: P3.52 (P52)
- new net GPIO_7: P3.44 (P44)
- new net GPIO_8: P3.45 (P45)
- new net GPIO_9: P3.48 (P48)
- new net SGPIO_0: P3.24 (P24)
- new net SGPIO_1: P3.25 (P25)
- new net SGPIO_2: P3.28 (P28)
- new net SGPIO_3: P3.29 (P29)
- new net SPGIO_4: P3.32 (P32)
Other:
- moved on the sheet: P1, P2

Commit message: Progress on board layout
Parts:
- J1, J2: symbol Conn_Coaxial -> conn:Conn_Coaxial
- P1, P2: symbol CONN_02X26 -> Header_Board-rescue:CONN_02X26
- P3: symbol CONN_02X30 -> Header_Board-rescue:CONN_02X30
- U1, U10, U12: symbol TAMP_1512GLN+ -> Header_Board-rescue:TAMP_1512GLN+
- U11, U13, U14, U15, U17, U18, U3, U4, U5, U6, U7, U9: symbol LAT -> Header_Board-rescue:LAT
- U16, U2, U8: symbol CBP-1400E+ -> Header_Board-rescue:CBP-1400E+
Connections:
- net GPIO_11 is gone; now on net GND: P3.52 (P52)
- net GPIO_7 is gone; now on net GND: P3.44 (P44)
- net GPIO_9 is gone; now on net GND: P3.48 (P48)
- net SGPIO_0 is gone; now on net GND: P3.24 (P24)
- net SGPIO_2 is gone; now on net GND: P3.28 (P28)
- net SPGIO_4 is gone; now on net GND: P3.32 (P32)
- net +3V3: no longer P3.11 (P11), P3.14 (P14), P3.2 (P2), P3.33 (P33), P3.36 (P36), P3.53 (P53), P3.56 (P56)
- net +5V: now also P3.33 (P33), P3.34 (P34), P3.37 (P37), P3.38 (P38); no longer P3.3 (P3), P3.57 (P57)
- net GND: now also P3.11 (P11), P3.15 (P15), P3.19 (P19), P3.2 (P2), P3.3 (P3), P3.36 (P36), P3.40 (P40), P3.56 (P56), P3.60 (P60), P3.7 (P7); no longer P3.13 (P13), P3.17 (P17), P3.26 (P26), P3.30 (P30), P3.34 (P34), P3.38 (P38), P3.42 (P42), P3.46 (P46), P3.5 (P5), P3.50 (P50), P3.54 (P54), P3.58 (P58), P3.9 (P9)
- net SPI2_MISO: no longer P3.15 (P15)
- net SPI2_MOSI: no longer P3.18 (P18)
- net SPI2_SCK: no longer P3.19 (P19)
- net SYS_SCL: no longer P3.7 (P7)
- net SYS_SDA: no longer P3.10 (P10)
- net SYS_SPI_MISO: no longer P3.37 (P37)
- net SYS_SPI_MOSI: no longer P3.40 (P40)
- net SYS_SPI_SCK: no longer P3.41 (P41)
- net +12V: no longer names the net of P3.6 (P6)
- net +12V: no longer P3.60 (P60)
- net GPIO_10: no longer names the net of P3.49 (P49)
- net GPIO_8: no longer names the net of P3.45 (P45)
- net SGPIO_1: no longer names the net of P3.25 (P25)
- net SGPIO_3: no longer names the net of P3.29 (P29)
Other:
- note added: "Cardedge Connector"
- moved on the sheet: J1, J2, P1, U1, U10, U11, U12, U13, U14, U15, U16, U17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
