File: LNA_Board.sch (KiCad schematic (older format))
At the start: 23 parts, among them J1 Conn_Coaxial, J2 Conn_Coaxial, P1 CONN_02X26, P2 CONN_02X26, P3 CONN_02X30, U1 TAMP_1512GLN+, U10 TAMP_1512GLN+, U11 LAT, U12 TAMP_1512GLN+, U13 LAT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

Commit message: Project rename
Renamed key files to better reflect what this board is, which is the LNA board for the SDR Radiometer.
Parts:
- J1, J2: symbol conn:Conn_Coaxial -> LNA_Board-rescue:Conn_Coaxial-conn
- P1, P2: symbol Header_Board-rescue:CONN_02X26 -> LNA_Board-rescue:CONN_02X26-Header_Board-rescue
- P3: symbol Header_Board-rescue:CONN_02X30 -> LNA_Board-rescue:CONN_02X30-Header_Board-rescue
- U1, U10, U12: symbol Header_Board-rescue:TAMP_1512GLN+ -> LNA_Board-rescue:TAMP_1512GLN+-Header_Board-rescue
- U11, U13, U14, U15, U17, U18, U3, U4, U5, U6, U7, U9: symbol Header_Board-rescue:LAT -> LNA_Board-rescue:LAT-Header_Board-rescue
- U16, U2, U8: symbol Header_Board-rescue:CBP-1400E+ -> LNA_Board-rescue:CBP-1400E+-Header_Board-rescue
Changed lines of the file:
@@
 EESchema Schematic File Version 4
-LIBS:Header_Board-cache
-EELAYER 26 0
+LIBS:LNA_Board-cache
+EELAYER 29 0
 EELAYER END
 $Descr A4 11693 8268
@@
 $EndDescr
 $Comp
-L Header_Board-rescue:CONN_02X26 P1
+L LNA_Board-rescue:CONN_02X26-Header_Board-rescue P1
 U 1 1 5AF36949
 P 5650 2100
@@
 $EndComp
 $Comp
-L Header_Board-rescue:CONN_02X26 P2
+L LNA_Board-rescue:CONN_02X26-Header_Board-rescue P2
 U 1 1 5AF3698C
 P 7650 2100
@@
 $EndComp
 $Comp
-L Header_Board-rescue:CONN_02X30 P3
+L LNA_Board-rescue:CONN_02X30-Header_Board-rescue P3
 U 1 1 5B16E67A
 P 9900 2250
@@
 $EndComp
 $Comp
-L conn:Conn_Coaxial J1
+L LNA_Board-rescue:Conn_Coaxial-conn J1
 U 1 1 5B4CFF90
 P 1100 1950
@@
 $EndComp
 $Comp
-L conn:Conn_Coaxial J2
+L LNA_Board-rescue:Conn_Coaxial-conn J2
 U 1 1 5B4CFFD6
 P 2350 6050
@@
 $EndComp
 $Comp
-L Header_Board-rescue:LAT U14
+L LNA_Board-rescue:LAT-Header_Board-rescue U14
 U 1 1 5B4DFEB1
 P 4200 2900
@@
 $EndComp
 $Comp
-L Header_Board-rescue:LAT U4
+L LNA_Board-rescue:LAT-Header_Board-rescue U4
 U 1 1 5B4DFEDE
 P 2400 3200
@@
 $EndComp
 $Comp
-L Header_Board-rescue:LAT U3
+L LNA_Board-rescue:LAT-Header_Board-rescue U3
 U 1 1 5B4DFF08
 P 2150 3200
@@
 $EndComp
 $Comp
-L Header_Board-rescue:LAT U5
+L LNA_Board-rescue:LAT-Header_Board-rescue U5
 U 1 1 5B4DFF31
 P 2400 4550
@@
 $EndComp
 $Comp
-L Header_Board-rescue:LAT U6
+L LNA_Board-rescue:LAT-Header_Board-rescue U6
 U 1 1 5B4DFF5D
 P 2700 4550
@@
 $EndComp
 $Comp
-L Header_Board-rescue:LAT U7
+L LNA_Board-rescue:LAT-Header_Board-rescue U7
 U 1 1 5B4DFF8C
 P 3000 4550
@@
 $EndComp
 $Comp
-L Header_Board-rescue:LAT U9
+L LNA_Board-rescue:LAT-Header_Board-rescue U9
 U 1 1 5B4DFFBF
 P 3350 4550
@@
 $EndComp
 $Comp
-L Header_Board-rescue:LAT U11
+L LNA_Board-rescue:LAT-Header_Board-rescue U11
 U 1 1 5B4DFFF4
 P 3700 4550
@@
 $EndComp
 $Comp
-L Header_Board-rescue:LAT U13
+L LNA_Board-rescue:LAT-Header_Board-rescue U13
 U 1 1 5B4E002E
 P 4050 4550
@@
 $EndComp
 $Comp
-L Header_Board-rescue:LAT U18
+L LNA_Board-rescue:LAT-Header_Board-rescue U18
 U 1 1 5B4E006B
 P 5650 5650
@@
 $EndComp
 $Comp
-L Header_Board-rescue:LAT U17
+L LNA_Board-rescue:LAT-Header_Board-rescue U17
 U 1 1 5B4E00A9
 P 5300 6000
@@
 $EndComp
 $Comp
-L Header_Board-rescue:LAT U15
+L LNA_Board-rescue:LAT-Header_Board-rescue U15
 U 1 1 5B4E00EA
 P 4950 6050
@@
 $EndComp
 $Comp
-L Header_Board-rescue:CBP-1400E+ U2
+L LNA_Board-rescue:CBP-1400E+-Header_Board-rescue U2
 U 1 1 5B4E0132
 P 1900 2050
@@
 $EndComp
 $Comp
-L Header_Board-rescue:CBP-1400E+ U8
+L LNA_Board-rescue:CBP-1400E+-Header_Board-rescue U8
 U 1 1 5B4E0189
 P 3250 3200
@@
 $EndComp
 $Comp
-L Header_Board-rescue:CBP-1400E+ U16
+L LNA_Board-rescue:CBP-1400E+-Header_Board-rescue U16
 U 1 1 5B4E01DB
 P 5000 4750
@@
 $EndComp
 $Comp
-L Header_Board-rescue:TAMP_1512GLN+ U10
+L LNA_Board-rescue:TAMP_1512GLN+-Header_Board-rescue U10
 U 1 1 5B4E0248
 P 3500 1950
@@
 $EndComp
 $Comp
-L Header_Board-rescue:TAMP_1512GLN+ U1
+L LNA_Board-rescue:TAMP_1512GLN+-Header_Board-rescue U1
 U 1 1 5B4E02B5
 P 1400 4600
@@
 $EndComp
 $Comp
-L Header_Board-rescue:TAMP_1512GLN+ U12
+L LNA_Board-rescue:TAMP_1512GLN+-Header_Board-rescue U12
 U 1 1 5B4E030F
 P 3800 6050
